File: Hardware/PCB.brd (EAGLE design)
At the start: 170.6 x 111.2 mm, 103 parts, among them IC1 BD5229G-TR, IC4 XC6220A331MR-G, J1 FH34SRJ-24S-0.5SH_99_, J2 SAMACSYS_PARTS_USB4110-GF-A, J3 QWIIC_RIGHT_ANGLE, J4 112A-TAAR-R03_ATTEND, Q1 20V/4.2A/52mΩ/1.4W, Q2 20V/4.2A/52mΩ/1.4W, Q3 SI1308EDL-T1-GE3, U1 W25Q512JVEIQ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

Commit message: Fix #5, Fix #11
Parts:
- C1, C10, C2, C5, C6, C8, C_DELAY, EPD_C1, EPD_C10, EPD_C11, EPD_C12, EPD_C2, EPD_C5, EPD_C6, EPD_C7, EPD_C8, EPD_C9: device DeskAssistant v19 v1:ESP32_WROVER_EAGLE-LTSPICE_C0402 -> DeskAssistant v19 v1:EAGLE-LTSPICE_C0402
